Commit message: Added gazebo control

File: description/robot_core.xacro (robot description, xacro)
@@ -44,4 +44,7 @@
         </xacro:inertial_box>
     </link>
+    <gazebo reference="chassis">
+        <material>Gazebo/Black</material>
+    </gazebo>
     <!-- LEFT WHEEL LINK -->
     <joint name="left_wheel_joint" type="continuous">
@@ -67,4 +70,7 @@
         </xacro:inertial_cylinder>
     </link>
+    <gazebo reference="left_wheel">
+        <material>Gazebo/Red</material>
+    </gazebo>
     <!-- RIGHT WHEEL LINK -->
     <joint name="right_wheel_joint" type="continuous">
@@ -90,4 +96,7 @@
         </xacro:inertial_cylinder>
     </link>
+    <gazebo reference="right_wheel">
+        <material>Gazebo/Red</material>
+    </gazebo>
     <!-- BACK RIGHT CASTER WHEEL (TANK TREAD WHEELS) LINK -->
     <joint name="back_right_caster_wheel_joint" type="fixed">
@@ -112,4 +121,9 @@
         </xacro:inertial_sphere>
     </link>
+    <gazebo reference="br_caster_wheel">
+        <material>Gazebo/Orange</material>
+        <mu1 value="0.0001"/>
+        <mu2 value="0.0001"/>
+    </gazebo>
     <!-- BACK LEFT CASTER WHEEL (TANK TREAD WHEELS) LINK -->
     <joint name="back_left_caster_wheel_joint" type="fixed">
@@ -134,4 +148,9 @@
         </xacro:inertial_sphere>
     </link>
+    <gazebo reference="bl_caster_wheel">
+        <material>Gazebo/Orange</material>
+        <mu1 value="0.0001"/>
+        <mu2 value="0.0001"/>
+    </gazebo>
     <!-- FRONT RIGHT CASTER WHEEL (TANK TREAD WHEELS) LINK -->
     <joint name="front_right_caster_wheel_joint" type="fixed">
@@ -156,4 +175,9 @@
         </xacro:inertial_sphere>
     </link>
+    <gazebo reference="fr_caster_wheel">
+        <material>Gazebo/Orange</material>
+        <mu1 value="0.0001"/>
+        <mu2 value="0.0001"/>
+    </gazebo>
     <!-- FRONT LEFT CASTER WHEEL (TANK TREAD WHEELS) LINK -->
     <joint name="front_left_caster_wheel_joint" type="fixed">
@@ -178,3 +202,8 @@
         </xacro:inertial_sphere>
     </link>
+    <gazebo reference="fl_caster_wheel">
+        <material>Gazebo/Orange</material>
+        <mu1 value="0.0001"/>
+        <mu2 value="0.0001"/>
+    </gazebo>
 </robot>
